Commit message: improved some dynamic parameters

File: robotis_humanoid_description/urdf/robotis_humanoid.inertia.xacro (robot description, xacro)
@@ -6,3 +6,39 @@
         <inertia ixx="1.0" ixy="0.0" ixz="0.0" iyy="1.0" iyz="0.0" izz="1.0" />
     </xacro:macro>
+  <xacro:macro name="inertial_cuboid_macro" params="mass x_length y_length z_length">
+    <inertial>
+      <mass value="${mass}" />
+      <origin xyz="0 0 0" />
+      <inertia ixx="${(1/12) * mass* (y_length*y_length+ z_length*z_length)}" ixy="0.0" ixz="0.0"
+               iyy="${(1/12) * mass* (x_length*x_length+ z_length*z_length)}" iyz="0.0"
+               izz="${(1/12) * mass* (x_length*x_length+ y_length*y_length)}" />
+    </inertial>
+  </xacro:macro>
+  <xacro:macro name="inertial_cuboid_with_pose_macro" params="mass x_length y_length z_length *origin">
+    <inertial>
+      <insert_block name="origin"/>
+      <mass value="${mass}" />
+      <inertia ixx="${(1/12) * mass* (y_length*y_length+ z_length*z_length)}" ixy="0.0" ixz="0.0"
+               iyy="${(1/12) * mass* (x_length*x_length+ z_length*z_length)}" iyz="0.0"
+               izz="${(1/12) * mass* (x_length*x_length+ y_length*y_length)}" />
+    </inertial>
+  </xacro:macro>
+  <xacro:macro name="inertial_sphere_macro" params="mass diameter">
+    <inertial>
+      <mass value="${mass}" />
+      <origin xyz="0 0 0" />
+      <inertia ixx="${(2/5) * mass* ( (diameter*0.5)) * (diameter*0.5))}" ixy="0.0" ixz="0.0"
+               iyy="${(2/5) * mass* ( (diameter*0.5)) * (diameter*0.5))}" iyz="0.0"
+               izz="${(2/5) * mass* ( (diameter*0.5)) * (diameter*0.5))}" />
+    </inertial>
+  </xacro:macro>
+  <xacro:macro name="inertial_sphere_with_pose_macro" params="mass diameter *origin">
+    <inertial>
+      <insert_block name="origin"/>
+      <mass value="${mass}" />
+      <inertia ixx="${(2/5) * mass* ( (diameter*0.5)) * (diameter*0.5))}" ixy="0.0" ixz="0.0"
+               iyy="${(2/5) * mass* ( (diameter*0.5)) * (diameter*0.5))}" iyz="0.0"
+               izz="${(2/5) * mass* ( (diameter*0.5)) * (diameter*0.5))}" />
+    </inertial>
+  </xacro:macro>
 </robot>

File: robotis_humanoid_description/urdf/robotis_humanoid.structure.arm.xacro (robot description, xacro)
@@ -10,5 +10,5 @@
           <child link="l_arm_sh_p1_link"/>
           <limit velocity="6.5" effort="1000" lower="${-pi*0.5}" upper="${pi*0.5}" />
-          <dynamics damping="0.1" friction="0.0" />
+          <dynamics damping="0.1" friction="0.1" />
         </joint>
         <xacro:insert_transmission name="l_arm_sh_p1" />
@@ -42,5 +42,5 @@
           <child link="l_arm_sh_r_link"/>
           <limit velocity="6.5" effort="1000" lower="${-pi*0.3}" upper="${pi*0.5}" />
-          <dynamics damping="0.1" friction="0.0" />
+          <dynamics damping="0.1" friction="0.1" />
         </joint>
         <xacro:insert_transmission name="l_arm_sh_r" />
@@ -74,5 +74,5 @@
           <child link="l_arm_sh_p2_link"/>
           <limit velocity="6.5" effort="1000" lower="${-pi*0.5}" upper="${pi*0.5}" />
-          <dynamics damping="0.1" friction="0.0" />
+          <dynamics damping="0.1" friction="0.1" />
         </joint>
         <xacro:insert_transmission name="l_arm_sh_p2" />
@@ -106,5 +106,5 @@
           <child link="l_arm_el_y_link"/>
           <limit velocity="6.5" effort="1000" lower="${-pi*0.4}" upper="${pi*0.4}" />
-          <dynamics damping="0.1" friction="0.0" />
+          <dynamics damping="0.1" friction="0.1" />
         </joint>
         <xacro:insert_transmission name="l_arm_el_y" />
@@ -138,5 +138,5 @@
           <child link="l_arm_wr_r_link"/>
           <limit velocity="6.5" effort="1000" lower="${-pi*0.5}" upper="${pi*0.5}" />
-          <dynamics damping="0.1" friction="0.0" />
+          <dynamics damping="0.1" friction="0.1" />
         </joint>
         <xacro:insert_transmission name="l_arm_wr_r" />
@@ -170,5 +170,5 @@
           <child link="l_arm_wr_y_link"/>
           <limit velocity="6.5" effort="1000" lower="${-pi*0.45}" upper="${pi*0.45}" />
-          <dynamics damping="0.1" friction="0.0" />
+          <dynamics damping="0.1" friction="0.1" />
         </joint>
         <xacro:insert_transmission name="l_arm_wr_y" />
@@ -202,5 +202,5 @@
           <child link="l_arm_wr_p_link"/>
           <limit velocity="6.5" effort="1000" lower="${-pi*0.45}" upper="${pi*0.45}" />
-          <dynamics damping="0.1" friction="0.0" />
+          <dynamics damping="0.1" friction="0.1" />
         </joint>
         <xacro:insert_transmission name="l_arm_wr_p" />
@@ -234,5 +234,5 @@
           <child link="l_arm_grip_link"/>
           <limit velocity="6.5" effort="1000" lower="${-pi*0.45}" upper="${pi*0.45}" />
-          <dynamics damping="0.1" friction="0.0" />
+          <dynamics damping="0.1" friction="0.1" />
         </joint>
         <xacro:insert_transmission name="l_arm_grip" />
@@ -266,5 +266,5 @@
           <child link="l_arm_grip_1_link"/>
           <limit velocity="6.5" effort="1000" lower="${-pi*0.45}" upper="${pi*0.45}" />
-          <dynamics damping="0.1" friction="0.0" />
+          <dynamics damping="0.1" friction="0.1" />
         </joint>
         <xacro:insert_transmission name="l_arm_grip_1" />
@@ -315,5 +315,5 @@
       	    <origin xyz="0.0 0.0 0.0" rpy="0 0 0"/>
       	    <mass value="0.001"/>
-      	    <!--inertia ixx="1.0" ixy="0.0" ixz="0.0" iyy="1.0" iyz="0.0" izz="1.0" /-->
+      	    <inertia ixx="0.00001" ixy="0.0" ixz="0.0" iyy="0.00001" iyz="0.0" izz="0.00001" />
     	  </inertial>
         </link>
@@ -327,5 +327,5 @@
           <child link="r_arm_sh_p1_link"/>
           <limit velocity="6.5" effort="1000" lower="${-pi*0.5}" upper="${pi*0.5}" />
-          <dynamics damping="0.1" friction="0.0" />
+          <dynamics damping="0.1" friction="0.1" />
         </joint>
         <xacro:insert_transmission name="r_arm_sh_p1" />
@@ -359,5 +359,5 @@
           <child link="r_arm_sh_r_link"/>
           <limit velocity="6.5" effort="1000" lower="${-pi*0.5}" upper="${pi*0.3}" />
-          <dynamics damping="0.1" friction="0.0" />
+          <dynamics damping="0.1" friction="0.1" />
         </joint>
         <xacro:insert_transmission name="r_arm_sh_r" />
@@ -391,5 +391,5 @@
           <child link="r_arm_sh_p2_link"/>
           <limit velocity="6.5" effort="1000" lower="${-pi*0.5}" upper="${pi*0.5}" />
-          <dynamics damping="0.1" friction="0.0" />
+          <dynamics damping="0.1" friction="0.1" />
         </joint>
         <xacro:insert_transmission name="r_arm_sh_p2" />
@@ -423,5 +423,5 @@
           <child link="r_arm_el_y_link"/>
           <limit velocity="6.5" effort="1000" lower="${-pi*0.4}" upper="${pi*0.4}" />
-          <dynamics damping="0.1" friction="0.0" />
+          <dynamics damping="0.1" friction="0.1" />
         </joint>
         <xacro:insert_transmission name="r_arm_el_y" />
@@ -455,5 +455,5 @@
           <child link="r_arm_wr_r_link"/>
           <limit velocity="6.5" effort="1000" lower="${-pi*0.5}" upper="${pi*0.5}" />
-          <dynamics damping="0.1" friction="0.0" />
+          <dynamics damping="0.1" friction="0.1" />
         </joint>
         <xacro:insert_transmission name="r_arm_wr_r" />
@@ -487,5 +487,5 @@
           <child link="r_arm_wr_y_link"/>
           <limit velocity="6.5" effort="1000" lower="${-pi*0.45}" upper="${pi*0.45}" />
-          <dynamics damping="0.1" friction="0.0" />
+          <dynamics damping="0.1" friction="0.1" />
         </joint>
         <xacro:insert_transmission name="r_arm_wr_y" />
@@ -519,5 +519,5 @@
           <child link="r_arm_wr_p_link"/>
           <limit velocity="6.5" effort="1000" lower="${-pi*0.45}" upper="${pi*0.45}" />
-          <dynamics damping="0.1" friction="0.0" />
+          <dynamics damping="0.1" friction="0.1" />
         </joint>
         <xacro:insert_transmission name="r_arm_wr_p" />
@@ -551,5 +551,5 @@
           <child link="r_arm_grip_link"/>
           <limit velocity="6.5" effort="1000" lower="${-pi*0.45}" upper="${pi*0.45}" />
-          <dynamics damping="0.1" friction="0.0" />
+          <dynamics damping="0.1" friction="0.1" />
         </joint>
         <xacro:insert_transmission name="r_arm_grip" />
@@ -583,5 +583,5 @@
           <child link="r_arm_grip_1_link"/>
           <limit velocity="6.5" effort="1000" lower="${-pi*0.45}" upper="${pi*0.45}" />
-          <dynamics damping="0.1" friction="0.0" />
+          <dynamics damping="0.1" friction="0.1" />
         </joint>
         <xacro:insert_transmission name="r_arm_grip_1" />
@@ -632,5 +632,5 @@
       	    <origin xyz="0.0 0.0 0.0" rpy="0 0 0"/>
       	    <mass value="0.001"/>
-      	    <!--inertia ixx="1.0" ixy="0.0" ixz="0.0" iyy="1.0" iyz="0.0" izz="1.0" /-->
+      	    <inertia ixx="0.00001" ixy="0.0" ixz="0.0" iyy="0.00001" iyz="0.0" izz="0.00001" />
     	  </inertial>
         </link>

File: robotis_humanoid_description/urdf/robotis_humanoid.structure.head.xacro (robot description, xacro)
@@ -10,5 +10,5 @@
           <child link="head_y_link"/>
           <limit velocity="6.5" effort="1000" lower="${-pi*0.5}" upper="${pi*0.5}" />
-          <dynamics damping="0.1" friction="0.0" />
+          <dynamics damping="0.1" friction="0.1" />
         </joint>
         <xacro:insert_transmission name="head_y" />
@@ -28,9 +28,5 @@
       	    <material name="grey"/>
     	  </visual>
-          <inertial>
-      	    <origin xyz="0.0 0.0 0.0" rpy="0 0 0"/>
-      	    <mass value="1.0"/>
-      	    <inertia ixx="1.0" ixy="0.0" ixz="0.0" iyy="1.0" iyz="0.0" izz="1.0" />
-    	  </inertial>
+          <xacro:inertial_cuboid_macro mass="0.2" x_length="0.040" y_length="0.100" z_length="0.050" />
         </link>
 	<!-- head pitch joint -->
@@ -41,5 +37,5 @@
           <child link="head_p_link"/>
           <limit velocity="6.5" effort="1000" lower="${-pi*0.5}" upper="${pi*0.5}" />
-          <dynamics damping="0.1" friction="0.0" />
+          <dynamics damping="0.1" friction="0.1" />
         </joint>
         <xacro:insert_transmission name="head_p" />
@@ -59,9 +55,7 @@
       	    <material name="grey"/>
     	  </visual>
-          <inertial>
-      	    <origin xyz="0.0 0.0 0.0" rpy="0 0 0"/>
-      	    <mass value="1.0"/>
-      	    <inertia ixx="1.0" ixy="0.0" ixz="0.0" iyy="1.0" iyz="0.0" izz="1.0" />
-    	  </inertial>
+          <xacro:inertial_cuboid_with_pose_macro mass="1.0" x_length="0.110" y_length="0.130" z_length="0.150">
+	    <origin xyz="0 0.050 0.050" rpy="0 0 0"/>
+	  </xacro:inertial_cuboid_with_pose_macro>
         </link>
 	<!-- camera joint -->

File: robotis_humanoid_description/urdf/robotis_humanoid.structure.leg.xacro (robot description, xacro)
@@ -10,5 +10,5 @@
           <child link="l_leg_hip_y_link"/>
           <limit velocity="6.5" effort="1000" lower="${-pi*0.45}" upper="${pi*0.45}" />
-          <dynamics damping="0.1" friction="0.0" />
+          <dynamics damping="0.1" friction="0.1" />
         </joint>
         <xacro:insert_transmission name="l_leg_hip_y" />
@@ -42,5 +42,5 @@
           <child link="l_leg_hip_r_link"/>
           <limit velocity="6.5" effort="1000" lower="${-pi*0.2}" upper="${pi*0.3}" />
-          <dynamics damping="0.1" friction="0.0" />
+          <dynamics damping="0.1" friction="0.1" />
         </joint>
         <xacro:insert_transmission name="l_leg_hip_r" />
@@ -74,5 +74,5 @@
           <child link="l_leg_hip_p_link"/>
           <limit velocity="6.5" effort="1000" lower="${-pi*0.4}" upper="${pi*0.4}" />
-          <dynamics damping="0.1" friction="0.0" />
+          <dynamics damping="0.1" friction="0.1" />
         </joint>
         <xacro:insert_transmission name="l_leg_hip_p" />
@@ -106,5 +106,5 @@
           <child link="l_leg_kn_p_link"/>
           <limit velocity="6.5" effort="1000" lower="${-pi*0.1}" upper="${pi*0.7}" />
-          <dynamics damping="0.1" friction="0.0" />
+          <dynamics damping="0.1" friction="0.1" />
         </joint>
         <xacro:insert_transmission name="l_leg_kn_p" />
@@ -138,5 +138,5 @@
           <child link="l_leg_an_p_link"/>
           <limit velocity="6.5" effort="1000" lower="${-pi*0.45}" upper="${pi*0.45}" />
-          <dynamics damping="0.1" friction="0.0" />
+          <dynamics damping="0.1" friction="0.1" />
         </joint>
         <xacro:insert_transmission name="l_leg_an_p" />
@@ -170,5 +170,5 @@
           <child link="l_leg_an_r_link"/>
           <limit velocity="6.5" effort="1000" lower="${-pi*0.5}" upper="${pi*0.4}" />
-          <dynamics damping="0.1" friction="0.0" />
+          <dynamics damping="0.1" friction="0.1" />
         </joint>
         <xacro:insert_transmission name="l_leg_an_r" />
@@ -232,5 +232,5 @@
           <child link="r_leg_hip_y_link"/>
           <limit velocity="6.5" effort="1000" lower="${-pi*0.45}" upper="${pi*0.45}" />
-          <dynamics damping="0.1" friction="0.0" />
+          <dynamics damping="0.1" friction="0.1" />
         </joint>
         <xacro:insert_transmission name="r_leg_hip_y" />
@@ -264,5 +264,5 @@
           <child link="r_leg_hip_r_link"/>
           <limit velocity="6.5" effort="1000" lower="${-pi*0.3}" upper="${pi*0.2}" />
-          <dynamics damping="0.1" friction="0.0" />
+          <dynamics damping="0.1" friction="0.1" />
         </joint>
         <xacro:insert_transmission name="r_leg_hip_r" />
@@ -296,5 +296,5 @@
           <child link="r_leg_hip_p_link"/>
           <limit velocity="6.5" effort="1000" lower="${-pi*0.4}" upper="${pi*0.4}" />
-          <dynamics damping="0.1" friction="0.0" />
+          <dynamics damping="0.1" friction="0.1" />
         </joint>
         <xacro:insert_transmission name="r_leg_hip_p" />
@@ -328,5 +328,5 @@
           <child link="r_leg_kn_p_link"/>
           <limit velocity="6.5" effort="1000" lower="${-pi*0.7}" upper="${pi*0.1}" />
-          <dynamics damping="0.1" friction="0.0" />
+          <dynamics damping="0.1" friction="0.1" />
         </joint>
         <xacro:insert_transmission name="r_leg_kn_p" />
@@ -360,5 +360,5 @@
           <child link="r_leg_an_p_link"/>
           <limit velocity="6.5" effort="1000" lower="${-pi*0.45}" upper="${pi*0.45}" />
-          <dynamics damping="0.1" friction="0.0" />
+          <dynamics damping="0.1" friction="0.1" />
         </joint>
         <xacro:insert_transmission name="r_leg_an_p" />
@@ -392,5 +392,5 @@
           <child link="r_leg_an_r_link"/>
           <limit velocity="6.5" effort="1000" lower="${-pi*0.45}" upper="${pi*0.45}" />
-          <dynamics damping="0.1" friction="0.0" />
+          <dynamics damping="0.1" friction="0.1" />
         </joint>
         <xacro:insert_transmission name="r_leg_an_r" />

File: robotis_humanoid_description/urdf/robotis_humanoid.xacro (robot description, xacro)
@@ -59,5 +59,5 @@
     <axis xyz="0 0 1"/>
     <limit velocity="6.5" effort="1000" lower="${-pi*0.6}" upper="${pi*0.6}" />
-    <dynamics damping="0.1" friction="0.0" />
+    <dynamics damping="0.1" friction="0.1" />
   </joint>
   <xacro:insert_transmission name="torso_y" />
