Commit message: changed inertial elements to calculated ones, fixed inertia of left_hip_yaw, temporarily added gazebo launch files for testing

File: robotis_humanoid_description/urdf/robotis_humanoid.structure.arm.xacro (robot description, xacro)
@@ -31,6 +31,6 @@
       	    <origin xyz="-0.003 0.020 -0.005" rpy="0 0 0"/>
       	    <mass value="0.194"/>
-      	    <inertia ixx="1.0" ixy="0.0" ixz="0.0" iyy="1.0" iyz="0.0" izz="1.0" />
-      	    <!--<inertia ixx="0.00018" ixy="0.0" ixz="0.0" iyy="0.00058" iyz="0.00004" izz="0.00057" />-->
+      	    <!--inertia ixx="1.0" ixy="0.0" ixz="0.0" iyy="1.0" iyz="0.0" izz="1.0" /-->
+      	    <inertia ixx="0.00018" ixy="0.0" ixz="0.0" iyy="0.00058" iyz="0.00004" izz="0.00057" />
     	  </inertial>
         </link>
@@ -63,6 +63,6 @@
       	    <origin xyz="-0.060 0.002 0.000" rpy="0 0 0"/>
       	    <mass value="0.875"/>
-            <inertia ixx="1.0" ixy="0.0" ixz="0.0" iyy="1.0" iyz="0.0" izz="1.0" />
-      	    <!--<inertia ixx="0.00043" ixy="0.0" ixz="0.0" iyy="0.00112" iyz="0.0" izz="0.00113" />-->
+            <!--inertia ixx="1.0" ixy="0.0" ixz="0.0" iyy="1.0" iyz="0.0" izz="1.0" /-->
+      	    <inertia ixx="0.00043" ixy="0.0" ixz="0.0" iyy="0.00112" iyz="0.0" izz="0.00113" />
     	  </inertial>
         </link>
@@ -95,6 +95,6 @@
       	    <origin xyz="0.000 0.073 0.000" rpy="0 0 0"/>
       	    <mass value="1.122"/>
-      	    <inertia ixx="1.0" ixy="0.0" ixz="0.0" iyy="1.0" iyz="0.0" izz="1.0" />
-      	    <!--<inertia ixx="0.00277" ixy="-0.00002" ixz="-0.00001" iyy="0.00090" iyz="-0.00004" izz="0.00255" />-->
+      	    <!--inertia ixx="1.0" ixy="0.0" ixz="0.0" iyy="1.0" iyz="0.0" izz="1.0" /-->
+      	    <inertia ixx="0.00277" ixy="-0.00002" ixz="-0.00001" iyy="0.00090" iyz="-0.00004" izz="0.00255" />
     	  </inertial>
         </link>
@@ -127,6 +127,6 @@
       	    <origin xyz="0.042 0.012 -0.058" rpy="0 0 0"/>
       	    <mass value="1.357"/>
-	    <inertia ixx="1.0" ixy="0.0" ixz="0.0" iyy="1.0" iyz="0.0" izz="1.0" />
-            <!--<inertia ixx="0.00152" ixy="-0.00100" ixz="-0.00006" iyy="0.00560" iyz="-0.00002" izz="0.00528" />-->
+	    <!--inertia ixx="1.0" ixy="0.0" ixz="0.0" iyy="1.0" iyz="0.0" izz="1.0" /-->
+            <inertia ixx="0.00152" ixy="-0.00100" ixz="-0.00006" iyy="0.00560" iyz="-0.00002" izz="0.00528" />
     	  </inertial>
         </link>
@@ -159,6 +159,6 @@
       	    <origin xyz="0.010 0.000 0.002" rpy="0 0 0"/>
       	    <mass value="0.087"/>
-            <inertia ixx="1.0" ixy="0.0" ixz="0.0" iyy="1.0" iyz="0.0" izz="1.0" />
-            <!--<inertia ixx="0.00012" ixy="0.0" ixz="0.0" iyy="0.00011" iyz="0.0" izz="0.00003" />-->
+            <!--inertia ixx="1.0" ixy="0.0" ixz="0.0" iyy="1.0" iyz="0.0" izz="1.0" /-->
+            <inertia ixx="0.00012" ixy="0.0" ixz="0.0" iyy="0.00011" iyz="0.0" izz="0.00003" />
     	  </inertial>
         </link>
@@ -191,6 +191,6 @@
       	    <origin xyz="0.023 0.001 -0.046" rpy="0 0 0"/>
       	    <mass value="0.768"/>
-      	    <inertia ixx="1.0" ixy="0.0" ixz="0.0" iyy="1.0" iyz="0.0" izz="1.0" />
-            <!--<inertia ixx="0.00059" ixy="-0.00002" ixz="-0.00002" iyy="0.00078" iyz="0.0" izz="0.00078" />-->
+      	    <!--inertia ixx="1.0" ixy="0.0" ixz="0.0" iyy="1.0" iyz="0.0" izz="1.0" /-->
+            <inertia ixx="0.00059" ixy="-0.00002" ixz="-0.00002" iyy="0.00078" iyz="0.0" izz="0.00078" />
     	  </inertial>
         </link>
@@ -223,6 +223,6 @@
       	    <origin xyz="0.065 0.045 0.000" rpy="0 0 0"/>
       	    <mass value="0.565"/>
-      	    <inertia ixx="1.0" ixy="0.0" ixz="0.0" iyy="1.0" iyz="0.0" izz="1.0" />
-            <!--<inertia ixx="0.00047" ixy="-0.00001" ixz="0.0" iyy="0.00042" iyz="0.0" izz="0.00058" />-->
+      	    <!--inertia ixx="1.0" ixy="0.0" ixz="0.0" iyy="1.0" iyz="0.0" izz="1.0" /-->
+            <inertia ixx="0.00047" ixy="-0.00001" ixz="0.0" iyy="0.00042" iyz="0.0" izz="0.00058" />
     	  </inertial>
         </link>
@@ -255,6 +255,6 @@
       	    <origin xyz="0.031 0.014 0.000" rpy="0 0 0"/>
       	    <mass value="0.013"/>
-      	    <inertia ixx="1.0" ixy="0.0" ixz="0.0" iyy="1.0" iyz="0.0" izz="1.0" />
-            <!--<inertia ixx="0.0" ixy="0.0" ixz="0.0" iyy="0.00001" iyz="0.0" izz="0.00001" />-->
+      	    <!--inertia ixx="1.0" ixy="0.0" ixz="0.0" iyy="1.0" iyz="0.0" izz="1.0" /-->
+            <inertia ixx="0.0" ixy="0.0" ixz="0.0" iyy="0.00001" iyz="0.0" izz="0.00001" />
     	  </inertial>
         </link>
@@ -287,6 +287,6 @@
       	    <origin xyz="0.031 -0.014 0.000" rpy="0 0 0"/>
       	    <mass value="0.013"/>
-      	    <inertia ixx="1.0" ixy="0.0" ixz="0.0" iyy="1.0" iyz="0.0" izz="1.0" />
-            <!--<inertia ixx="0.0" ixy="0.0" ixz="0.0" iyy="0.00001" iyz="0.0" izz="0.00001" />-->
+      	    <!--inertia ixx="1.0" ixy="0.0" ixz="0.0" iyy="1.0" iyz="0.0" izz="1.0" /-->
+            <inertia ixx="0.0" ixy="0.0" ixz="0.0" iyy="0.00001" iyz="0.0" izz="0.00001" />
     	  </inertial>
         </link>
@@ -315,5 +315,5 @@
       	    <origin xyz="0.0 0.0 0.0" rpy="0 0 0"/>
       	    <mass value="0.001"/>
-      	    <inertia ixx="1.0" ixy="0.0" ixz="0.0" iyy="1.0" iyz="0.0" izz="1.0" />
+      	    <!--inertia ixx="1.0" ixy="0.0" ixz="0.0" iyy="1.0" iyz="0.0" izz="1.0" /-->
     	  </inertial>
         </link>
@@ -348,6 +348,6 @@
       	    <origin xyz="-0.003 -0.020 -0.005" rpy="0 0 0"/>
       	    <mass value="0.194"/>
-      	    <inertia ixx="1.0" ixy="0.0" ixz="0.0" iyy="1.0" iyz="0.0" izz="1.0" />
-            <!--<inertia ixx="0.00018" ixy="0.0" ixz="0.0" iyy="0.00058" iyz="-0.00004" izz="0.00057" />-->
+      	    <!--inertia ixx="1.0" ixy="0.0" ixz="0.0" iyy="1.0" iyz="0.0" izz="1.0" /-->
+            <inertia ixx="0.00018" ixy="0.0" ixz="0.0" iyy="0.00058" iyz="-0.00004" izz="0.00057" />
     	  </inertial>
         </link>
@@ -380,6 +380,6 @@
       	    <origin xyz="-0.060 -0.002 0.000" rpy="0 0 0"/>
       	    <mass value="0.875"/>
-      	    <inertia ixx="1.0" ixy="0.0" ixz="0.0" iyy="1.0" iyz="0.0" izz="1.0" />
-            <!--<inertia ixx="0.00043" ixy="0.0" ixz="0.0" iyy="0.00112" iyz="0.0" izz="0.00113" />-->
+      	    <!--inertia ixx="1.0" ixy="0.0" ixz="0.0" iyy="1.0" iyz="0.0" izz="1.0" /-->
+            <inertia ixx="0.00043" ixy="0.0" ixz="0.0" iyy="0.00112" iyz="0.0" izz="0.00113" />
     	  </inertial>
         </link>
@@ -412,6 +412,6 @@
       	    <origin xyz="0.000 -0.073 0.000" rpy="0 0 0"/>
       	    <mass value="1.122"/>
-      	    <inertia ixx="1.0" ixy="0.0" ixz="0.0" iyy="1.0" iyz="0.0" izz="1.0" />
-            <!--<inertia ixx="0.00277" ixy="0.00002" ixz="-0.00001" iyy="0.00090" iyz="0.00004" izz="0.00255" />-->
+      	    <!--inertia ixx="1.0" ixy="0.0" ixz="0.0" iyy="1.0" iyz="0.0" izz="1.0" /-->
+            <inertia ixx="0.00277" ixy="0.00002" ixz="-0.00001" iyy="0.00090" iyz="0.00004" izz="0.00255" />
     	  </inertial>
         </link>
@@ -444,6 +444,6 @@
       	    <origin xyz="0.042 -0.012 -0.058" rpy="0 0 0"/>
       	    <mass value="1.357"/>
-      	    <inertia ixx="1.0" ixy="0.0" ixz="0.0" iyy="1.0" iyz="0.0" izz="1.0" />
-            <!--<inertia ixx="0.00152" ixy="0.00100" ixz="-0.00006" iyy="0.00560" iyz="0.00002" izz="0.00528" />-->
+      	    <!--inertia ixx="1.0" ixy="0.0" ixz="0.0" iyy="1.0" iyz="0.0" izz="1.0" /-->
+            <inertia ixx="0.00152" ixy="0.00100" ixz="-0.00006" iyy="0.00560" iyz="0.00002" izz="0.00528" />
     	  </inertial>
         </link>
@@ -476,6 +476,6 @@
       	    <origin xyz="0.010 0.000 -0.002" rpy="0 0 0"/>
       	    <mass value="0.087"/>
-      	    <inertia ixx="1.0" ixy="0.0" ixz="0.0" iyy="1.0" iyz="0.0" izz="1.0" />
-            <!--<inertia ixx="0.00012" ixy="0.0" ixz="0.0" iyy="0.00011" iyz="0.0" izz="0.00003" />-->
+      	    <!--inertia ixx="1.0" ixy="0.0" ixz="0.0" iyy="1.0" iyz="0.0" izz="1.0" /-->
+            <inertia ixx="0.00012" ixy="0.0" ixz="0.0" iyy="0.00011" iyz="0.0" izz="0.00003" />
     	  </inertial>
         </link>
@@ -508,6 +508,6 @@
       	    <origin xyz="0.023 -0.001 -0.046" rpy="0 0 0"/>
       	    <mass value="0.768"/>
-      	    <inertia ixx="1.0" ixy="0.0" ixz="0.0" iyy="1.0" iyz="0.0" izz="1.0" />
-            <!--<inertia ixx="0.00059" ixy="0.00002" ixz="-0.00002" iyy="0.00078" iyz="0.0" izz="0.00078" />-->
+      	    <!--inertia ixx="1.0" ixy="0.0" ixz="0.0" iyy="1.0" iyz="0.0" izz="1.0" /-->
+            <inertia ixx="0.00059" ixy="0.00002" ixz="-0.00002" iyy="0.00078" iyz="0.0" izz="0.00078" />
     	  </inertial>
         </link>
@@ -540,6 +540,6 @@
       	    <origin xyz="0.065 -0.045 0.000" rpy="0 0 0"/>
       	    <mass value="0.565"/>
-      	    <inertia ixx="1.0" ixy="0.0" ixz="0.0" iyy="1.0" iyz="0.0" izz="1.0" />
-            <!--<inertia ixx="0.00047" ixy="0.00001" ixz="0.0" iyy="0.00042" iyz="0.0" izz="0.00058" />-->
+      	    <!--inertia ixx="1.0" ixy="0.0" ixz="0.0" iyy="1.0" iyz="0.0" izz="1.0" /-->
+            <inertia ixx="0.00047" ixy="0.00001" ixz="0.0" iyy="0.00042" iyz="0.0" izz="0.00058" />
     	  </inertial>
         </link>
@@ -572,6 +572,6 @@
       	    <origin xyz="0.031 -0.014 0.000" rpy="0 0 0"/>
       	    <mass value="0.013"/>
-      	    <inertia ixx="1.0" ixy="0.0" ixz="0.0" iyy="1.0" iyz="0.0" izz="1.0" />
-            <!--<inertia ixx="0.0" ixy="0.0" ixz="0.0" iyy="0.00001" iyz="0.0" izz="0.00001" />-->
+      	    <!--inertia ixx="1.0" ixy="0.0" ixz="0.0" iyy="1.0" iyz="0.0" izz="1.0" /-->
+            <inertia ixx="0.0" ixy="0.0" ixz="0.0" iyy="0.00001" iyz="0.0" izz="0.00001" />
     	  </inertial>
         </link>
@@ -604,6 +604,6 @@
       	    <origin xyz="0.031 0.014 0.000" rpy="0 0 0"/>
       	    <mass value="0.013"/>
-      	    <inertia ixx="1.0" ixy="0.0" ixz="0.0" iyy="1.0" iyz="0.0" izz="1.0" />
-            <!--<inertia ixx="0.0" ixy="0.0" ixz="0.0" iyy="0.00001" iyz="0.0" izz="0.00001" />-->
+      	    <!--inertia ixx="1.0" ixy="0.0" ixz="0.0" iyy="1.0" iyz="0.0" izz="1.0" /-->
+            <inertia ixx="0.0" ixy="0.0" ixz="0.0" iyy="0.00001" iyz="0.0" izz="0.00001" />
     	  </inertial>
         </link>
@@ -632,5 +632,5 @@
       	    <origin xyz="0.0 0.0 0.0" rpy="0 0 0"/>
       	    <mass value="0.001"/>
-      	    <inertia ixx="1.0" ixy="0.0" ixz="0.0" iyy="1.0" iyz="0.0" izz="1.0" />
+      	    <!--inertia ixx="1.0" ixy="0.0" ixz="0.0" iyy="1.0" iyz="0.0" izz="1.0" /-->
     	  </inertial>
         </link>

File: robotis_humanoid_description/urdf/robotis_humanoid.structure.leg.xacro (robot description, xacro)
@@ -29,8 +29,8 @@
     	  </visual>
           <inertial>
-      	    <origin xyz="0.012 0.000 -0.025" rpy="0 0 0"/>
+      	    <origin xyz="-0.012 0.000 -0.025" rpy="0 0 0"/>
       	    <mass value="0.243"/>
-      	    <inertia ixx="1.0" ixy="0.0" ixz="0.0" iyy="1.0" iyz="0.0" izz="1.0" />
-    	    <!-- <inertia ixx="0.00024" ixy="0.0" ixz="0.0" iyy="0.00101" iyz="0.0" izz="0.00092" /> -->
+      	    <!--inertia ixx="1.0" ixy="0.0" ixz="0.0" iyy="1.0" iyz="0.0" izz="1.0" /-->
+    	    <inertia ixx="0.00024" ixy="0.0" ixz="0.0" iyy="0.00101" iyz="0.0" izz="0.00092" />
 	  </inertial>
         </link>
@@ -63,6 +63,6 @@
       	    <origin xyz="-0.068 0.000 0.000" rpy="0 0 0"/>
       	    <mass value="1.045"/>
-      	    <inertia ixx="1.0" ixy="0.0" ixz="0.0" iyy="1.0" iyz="0.0" izz="1.0" />
-            <!-- <inertia ixx="0.00056" ixy="0.0" ixz="0.0" iyy="0.00168" iyz="0.0" izz="0.00171" /> -->
+      	    <!--inertia ixx="1.0" ixy="0.0" ixz="0.0" iyy="1.0" iyz="0.0" izz="1.0" /-->
+            <inertia ixx="0.00056" ixy="0.0" ixz="0.0" iyy="0.00168" iyz="0.0" izz="0.00171" />
     	  </inertial>
         </link>
@@ -95,6 +95,6 @@
       	    <origin xyz="0.022 -0.007 -0.168" rpy="0 0 0"/>
       	    <mass value="3.095"/>
-      	    <inertia ixx="1.0" ixy="0.0" ixz="0.0" iyy="1.0" iyz="0.0" izz="1.0" />
-            <!-- <inertia ixx="0.04328" ixy="0.00028" ixz="0.00288" iyy="0.04042" iyz="-0.00202" izz="0.00560" /> -->
+      	    <!--inertia ixx="1.0" ixy="0.0" ixz="0.0" iyy="1.0" iyz="0.0" izz="1.0" /-->
+            <inertia ixx="0.04328" ixy="0.00028" ixz="0.00288" iyy="0.04042" iyz="-0.00202" izz="0.00560" />
     	  </inertial>
         </link>
@@ -127,6 +127,6 @@
       	    <origin xyz="-0.002 -0.066 -0.183" rpy="0 0 0"/>
       	    <mass value="2.401"/>
-      	    <inertia ixx="1.0" ixy="0.0" ixz="0.0" iyy="1.0" iyz="0.0" izz="1.0" />
-            <!-- <inertia ixx="0.01971" ixy="0.00031" ixz="-0.00294" iyy="0.01687" iyz="0.00140" izz="0.00574" /> -->
+      	    <!--inertia ixx="1.0" ixy="0.0" ixz="0.0" iyy="1.0" iyz="0.0" izz="1.0" /-->
+            <inertia ixx="0.01971" ixy="0.00031" ixz="-0.00294" iyy="0.01687" iyz="0.00140" izz="0.00574" />
     	  </inertial>
         </link>
@@ -159,6 +159,6 @@
       	    <origin xyz="-0.011 -0.033 0.000" rpy="0 0 0"/>
       	    <mass value="1.045"/>
-      	    <inertia ixx="1.0" ixy="0.0" ixz="0.0" iyy="1.0" iyz="0.0" izz="1.0" />
-            <!-- <inertia ixx="0.00056" ixy="0.0" ixz="0.0" iyy="0.00168" iyz="0.0" izz="0.00171" /> -->
+      	    <!--inertia ixx="1.0" ixy="0.0" ixz="0.0" iyy="1.0" iyz="0.0" izz="1.0" /-->
+            <inertia ixx="0.00056" ixy="0.0" ixz="0.0" iyy="0.00168" iyz="0.0" izz="0.00171" />
     	  </inertial>
         </link>
@@ -191,6 +191,6 @@
       	    <origin xyz="-0.070 0.000 -0.048" rpy="0 0 0"/>
       	    <mass value="0.223"/>
-      	    <inertia ixx="1.0" ixy="0.0" ixz="0.0" iyy="1.0" iyz="0.0" izz="1.0" />
-            <!-- <inertia ixx="0.00022" ixy="0.0" ixz="-0.00001" iyy="0.00099" iyz="0.0" izz="0.00091" /> -->
+      	    <!--inertia ixx="1.0" ixy="0.0" ixz="0.0" iyy="1.0" iyz="0.0" izz="1.0" /-->
+            <inertia ixx="0.00022" ixy="0.0" ixz="-0.00001" iyy="0.00099" iyz="0.0" izz="0.00091" />
     	  </inertial>
         </link>
@@ -219,6 +219,6 @@
       	    <origin xyz="0.000 0.009 -0.013" rpy="0 0 0"/>
       	    <mass value="1.689"/>
-      	    <inertia ixx="1.0" ixy="0.0" ixz="0.0" iyy="1.0" iyz="0.0" izz="1.0" />
-            <!-- <inertia ixx="0.00219" ixy="0.0" ixz="0.0" iyy="0.00433" iyz="0.00011" izz="0.00609" /> -->
+      	    <!--inertia ixx="1.0" ixy="0.0" ixz="0.0" iyy="1.0" iyz="0.0" izz="1.0" /-->
+            <inertia ixx="0.00219" ixy="0.0" ixz="0.0" iyy="0.00433" iyz="0.00011" izz="0.00609" />
     	  </inertial>
         </link>
@@ -253,6 +253,6 @@
       	    <origin xyz="-0.012 0.000 -0.025" rpy="0 0 0"/>
       	    <mass value="0.243"/>
-      	    <inertia ixx="1.0" ixy="0.0" ixz="0.0" iyy="1.0" iyz="0.0" izz="1.0" />
-            <!-- <inertia ixx="0.00024" ixy="0.0" ixz="0.0" iyy="0.00101" iyz="0.0" izz="0.00092" /> -->
+      	    <!--inertia ixx="1.0" ixy="0.0" ixz="0.0" iyy="1.0" iyz="0.0" izz="1.0" /-->
+            <inertia ixx="0.00024" ixy="0.0" ixz="0.0" iyy="0.00101" iyz="0.0" izz="0.00092" />
     	  </inertial>
         </link>
@@ -285,6 +285,6 @@
       	    <origin xyz="-0.068 0.000 0.000" rpy="0 0 0"/>
       	    <mass value="1.045"/>
-      	    <inertia ixx="1.0" ixy="0.0" ixz="0.0" iyy="1.0" iyz="0.0" izz="1.0" />
-            <!-- <inertia ixx="0.00056" ixy="0.0" ixz="0.0" iyy="0.00168" iyz="0.0" izz="0.00171" /> -->
+      	    <!--inertia ixx="1.0" ixy="0.0" ixz="0.0" iyy="1.0" iyz="0.0" izz="1.0" /-->
+            <inertia ixx="0.00056" ixy="0.0" ixz="0.0" iyy="0.00168" iyz="0.0" izz="0.00171" />
     	  </inertial>
         </link>
@@ -317,6 +317,6 @@
       	    <origin xyz="0.022 0.007 -0.168" rpy="0 0 0"/>
       	    <mass value="3.095"/>
-      	    <inertia ixx="1.0" ixy="0.0" ixz="0.0" iyy="1.0" iyz="0.0" izz="1.0" />
-            <!-- <inertia ixx="0.04328" ixy="-0.00027" ixz="0.00286" iyy="0.04042" iyz="-0.00202" izz="0.00560" /> -->
+      	    <!--inertia ixx="1.0" ixy="0.0" ixz="0.0" iyy="1.0" iyz="0.0" izz="1.0" /-->
+            <inertia ixx="0.04328" ixy="-0.00027" ixz="0.00286" iyy="0.04042" iyz="-0.00202" izz="0.00560" />
     	  </inertial>
         </link>
@@ -349,6 +349,6 @@
       	    <origin xyz="-0.002 0.066 -0.183" rpy="0 0 0"/>
       	    <mass value="2.401"/>
-      	    <inertia ixx="1.0" ixy="0.0" ixz="0.0" iyy="1.0" iyz="0.0" izz="1.0" />
-            <!-- <inertia ixx="0.01971" ixy="-0.00031" ixz="-0.00294" iyy="0.01687" iyz="-0.00140" izz="0.00574" /> -->
+      	    <!--inertia ixx="1.0" ixy="0.0" ixz="0.0" iyy="1.0" iyz="0.0" izz="1.0" /-->
+            <inertia ixx="0.01971" ixy="-0.00031" ixz="-0.00294" iyy="0.01687" iyz="-0.00140" izz="0.00574" />
     	  </inertial>
         </link>
@@ -381,6 +381,6 @@
       	    <origin xyz="-0.011 0.033 0.000" rpy="0 0 0"/>
       	    <mass value="1.045"/>
-      	    <inertia ixx="1.0" ixy="0.0" ixz="0.0" iyy="1.0" iyz="0.0" izz="1.0" />
-            <!-- <inertia ixx="0.00056" ixy="0.0" ixz="0.0" iyy="0.00168" iyz="0.0" izz="0.00171" /> -->
+      	    <!--inertia ixx="1.0" ixy="0.0" ixz="0.0" iyy="1.0" iyz="0.0" izz="1.0" /-->
+            <inertia ixx="0.00056" ixy="0.0" ixz="0.0" iyy="0.00168" iyz="0.0" izz="0.00171" />
     	  </inertial>
         </link>
@@ -413,6 +413,6 @@
       	    <origin xyz="-0.070 0.000 -0.048" rpy="0 0 0"/>
       	    <mass value="0.223"/>
-      	    <inertia ixx="1.0" ixy="0.0" ixz="0.0" iyy="1.0" iyz="0.0" izz="1.0" />
-            <!-- <inertia ixx="0.00022" ixy="0.0" ixz="-0.00001" iyy="0.00099" iyz="0.0" izz="0.00091" /> -->
+      	    <!--inertia ixx="1.0" ixy="0.0" ixz="0.0" iyy="1.0" iyz="0.0" izz="1.0" /-->
+            <inertia ixx="0.00022" ixy="0.0" ixz="-0.00001" iyy="0.00099" iyz="0.0" izz="0.00091" />
     	  </inertial>
         </link>
@@ -441,6 +441,6 @@
       	    <origin xyz="0.000 -0.009 -0.013" rpy="0 0 0"/>
       	    <mass value="1.689"/>
-      	    <inertia ixx="1.0" ixy="0.0" ixz="0.0" iyy="1.0" iyz="0.0" izz="1.0" />
-            <!-- <inertia ixx="0.00219" ixy="0.0" ixz="0.0" iyy="0.00433" iyz="-0.00011" izz="0.00609" /> -->
+      	    <!--inertia ixx="1.0" ixy="0.0" ixz="0.0" iyy="1.0" iyz="0.0" izz="1.0" /-->
+            <inertia ixx="0.00219" ixy="0.0" ixz="0.0" iyy="0.00433" iyz="-0.00011" izz="0.00609" />
     	  </inertial>
         </link>

File: robotis_humanoid_description/urdf/robotis_humanoid.xacro (robot description, xacro)
@@ -48,6 +48,6 @@
       <origin xyz="-0.011 0.000 0.058" rpy="0 0 0"/>
       <mass value="6.869"/>
-      <inertia ixx="1.0" ixy="0.0" ixz="0.0" iyy="1.0" iyz="0.0" izz="1.0" />
-      <!--<inertia ixx="0.03603" ixy="0.0" ixz="0.00016" iyy="0.02210" iyz="0.0" izz="0.03830" />-->
+      <!--inertia ixx="1.0" ixy="0.0" ixz="0.0" iyy="1.0" iyz="0.0" izz="1.0" /-->
+      <inertia ixx="0.03603" ixy="0.0" ixz="0.00016" iyy="0.02210" iyz="0.0" izz="0.03830" />
     </inertial>
   </link>
@@ -80,5 +80,5 @@
       <origin xyz="-0.007 0.000 0.109" rpy="0 0 0"/>
       <mass value="5.383"/>
-      <inertia ixx="1.0" ixy="0.0" ixz="0.0" iyy="1.0" iyz="0.0" izz="1.0" />
+      <!--inertia ixx="1.0" ixy="0.0" ixz="0.0" iyy="1.0" iyz="0.0" izz="1.0" /-->
       <inertia ixx="0.04710" ixy="0.0" ixz="0.04710" iyy="0.02554" iyz="0.0" izz="0.03094" />
     </inertial>
