Commit message: added motor-models and transmission-names

File: robotis_humanoid_description/urdf/robotis_humanoid.structure.arm.xacro (robot description, xacro)
@@ -9,8 +9,9 @@
           <parent link="${parent}"/>
           <child link="l_arm_sh_p1_link"/>
-          <limit velocity="6.5" effort="1000" lower="${-pi*0.5}" upper="${pi*0.5}" />
-          <dynamics damping="0.1" friction="0.1" />
-        </joint>
-        <xacro:insert_transmission name="l_arm_sh_p1" />
+          <!--limit velocity="6.5" effort="1000" lower="${-pi*0.5}" upper="${pi*0.5}" />
+          <dynamics damping="0.1" friction="0.1" /-->
+	  <xacro:joint_medium_servo_limits_macro lower="${-pi*0.5}" upper="${pi*0.5}" />
+        </joint>
+        <xacro:effort_transmission name="l_arm_sh_p1" servo="H54-100-S500" />
 	<!-- left shoulder pitch 1 link -->
         <link name="l_arm_sh_p1_link">
@@ -41,8 +42,9 @@
           <parent link="l_arm_sh_p1_link"/>
           <child link="l_arm_sh_r_link"/>
-          <limit velocity="6.5" effort="1000" lower="${-pi*0.3}" upper="${pi*0.5}" />
-          <dynamics damping="0.1" friction="0.1" />
-        </joint>
-        <xacro:insert_transmission name="l_arm_sh_r" />
+          <!--limit velocity="6.5" effort="1000" lower="${-pi*0.3}" upper="${pi*0.5}" />
+          <dynamics damping="0.1" friction="0.1" /-->
+	  <xacro:joint_medium_servo_limits_macro lower="${-pi*0.3}" upper="${pi*0.5}" />
+        </joint>
+        <xacro:effort_transmission name="l_arm_sh_r" servo="H54-100-S500" />
 	<!-- left shoulder roll link -->
         <link name="l_arm_sh_r_link">
@@ -73,8 +75,9 @@
           <parent link="l_arm_sh_r_link"/>
           <child link="l_arm_sh_p2_link"/>
-          <limit velocity="6.5" effort="1000" lower="${-pi*0.5}" upper="${pi*0.5}" />
-          <dynamics damping="0.1" friction="0.1" />
-        </joint>
-        <xacro:insert_transmission name="l_arm_sh_p2" />
+          <!--limit velocity="6.5" effort="1000" lower="${-pi*0.5}" upper="${pi*0.5}" />
+          <dynamics damping="0.1" friction="0.1" /-->
+	  <xacro:joint_medium_servo_limits_macro lower="${-pi*0.5}" upper="${pi*0.5}" />
+        </joint>
+        <xacro:effort_transmission name="l_arm_sh_p2" servo="H54-100-S500" />
 	<!-- left shoulder pitch2 link -->
         <link name="l_arm_sh_p2_link">
@@ -105,8 +108,9 @@
           <parent link="l_arm_sh_p2_link"/>
           <child link="l_arm_el_y_link"/>
-          <limit velocity="6.5" effort="1000" lower="${-pi*0.4}" upper="${pi*0.4}" />
-          <dynamics damping="0.1" friction="0.1" />
-        </joint>
-        <xacro:insert_transmission name="l_arm_el_y" />
+          <!--limit velocity="6.5" effort="1000" lower="${-pi*0.4}" upper="${pi*0.4}" />
+          <dynamics damping="0.1" friction="0.1" /-->
+	  <xacro:joint_medium_servo_limits_macro lower="${-pi*0.4}" upper="${pi*0.4}" />
+        </joint>
+        <xacro:effort_transmission name="l_arm_el_y" servo="H54-100-S500" />
 	<!-- left elbow yaw link -->
         <link name="l_arm_el_y_link">
@@ -137,8 +141,9 @@
           <parent link="l_arm_el_y_link"/>
           <child link="l_arm_wr_r_link"/>
-          <limit velocity="6.5" effort="1000" lower="${-pi*0.5}" upper="${pi*0.5}" />
-          <dynamics damping="0.1" friction="0.1" />
-        </joint>
-        <xacro:insert_transmission name="l_arm_wr_r" />
+          <!--limit velocity="6.5" effort="1000" lower="${-pi*0.5}" upper="${pi*0.5}" />
+          <dynamics damping="0.1" friction="0.1" /-->
+	  <xacro:joint_small_servo_limits_macro lower="${-pi*0.5}" upper="${pi*0.5}" />
+        </joint>
+        <xacro:effort_transmission name="l_arm_wr_r" servo="H42-20-S300" />
 	<!-- left wrist roll link -->
         <link name="l_arm_wr_r_link">
@@ -169,8 +174,9 @@
           <parent link="l_arm_wr_r_link"/>
           <child link="l_arm_wr_y_link"/>
-          <limit velocity="6.5" effort="1000" lower="${-pi*0.45}" upper="${pi*0.45}" />
-          <dynamics damping="0.1" friction="0.1" />
-        </joint>
-        <xacro:insert_transmission name="l_arm_wr_y" />
+          <!--limit velocity="6.5" effort="1000" lower="${-pi*0.45}" upper="${pi*0.45}" />
+          <dynamics damping="0.1" friction="0.1" /-->
+	  <xacro:joint_small_servo_limits_macro lower="${-pi*0.45}" upper="${pi*0.45}" />
+        </joint>
+        <xacro:effort_transmission name="l_arm_wr_y" servo="H42-20-S300" />
 	<!-- left wrist yaw link -->
         <link name="l_arm_wr_y_link">
@@ -201,8 +207,9 @@
           <parent link="l_arm_wr_y_link"/>
           <child link="l_arm_wr_p_link"/>
-          <limit velocity="6.5" effort="1000" lower="${-pi*0.45}" upper="${pi*0.45}" />
-          <dynamics damping="0.1" friction="0.1" />
-        </joint>
-        <xacro:insert_transmission name="l_arm_wr_p" />
+          <!--limit velocity="6.5" effort="1000" lower="${-pi*0.45}" upper="${pi*0.45}" />
+          <dynamics damping="0.1" friction="0.1" /-->
+	  <xacro:joint_small_servo_limits_macro lower="${-pi*0.45}" upper="${pi*0.45}" />
+        </joint>
+        <xacro:effort_transmission name="l_arm_wr_p" servo="H42-20-S300" />
 	<!-- left wrist pitch link -->
         <link name="l_arm_wr_p_link">
@@ -233,8 +240,9 @@
           <parent link="l_arm_wr_p_link"/>
           <child link="l_arm_grip_link"/>
-          <limit velocity="6.5" effort="1000" lower="${-pi*0.45}" upper="${pi*0.45}" />
-          <dynamics damping="0.1" friction="0.1" />
-        </joint>
-        <xacro:insert_transmission name="l_arm_grip" />
+          <!--limit velocity="6.5" effort="1000" lower="${-pi*0.45}" upper="${pi*0.45}" />
+          <dynamics damping="0.1" friction="0.1" /-->
+	  <xacro:joint_small_servo_limits_macro lower="${-pi*0.45}" upper="${pi*0.45}" />
+        </joint>
+        <xacro:effort_transmission name="l_arm_grip" servo="H42-20-S300" />
 	<!-- left arm gripper link -->
         <link name="l_arm_grip_link">
@@ -265,8 +273,9 @@
           <parent link="l_arm_wr_p_link"/>
           <child link="l_arm_grip_1_link"/>
-          <limit velocity="6.5" effort="1000" lower="${-pi*0.45}" upper="${pi*0.45}" />
-          <dynamics damping="0.1" friction="0.1" />
-        </joint>
-        <xacro:insert_transmission name="l_arm_grip_1" />
+          <!--limit velocity="6.5" effort="1000" lower="${-pi*0.45}" upper="${pi*0.45}" />
+          <dynamics damping="0.1" friction="0.1" /-->
+	  <xacro:joint_small_servo_limits_macro lower="${-pi*0.45}" upper="${pi*0.45}" />
+        </joint>
+        <xacro:effort_transmission name="l_arm_grip_1" servo="H42-20-S300" />
 	<!-- left arm gripper 1 link -->
         <link name="l_arm_grip_1_link">
@@ -326,8 +335,9 @@
           <parent link="${parent}"/>
           <child link="r_arm_sh_p1_link"/>
-          <limit velocity="6.5" effort="1000" lower="${-pi*0.5}" upper="${pi*0.5}" />
-          <dynamics damping="0.1" friction="0.1" />
-        </joint>
-        <xacro:insert_transmission name="r_arm_sh_p1" />
+          <!--limit velocity="6.5" effort="1000" lower="${-pi*0.5}" upper="${pi*0.5}" />
+          <dynamics damping="0.1" friction="0.1" /-->
+	  <xacro:joint_medium_servo_limits_macro lower="${-pi*0.5}" upper="${pi*0.5}" />
+        </joint>
+        <xacro:effort_transmission name="r_arm_sh_p1" servo="H54-100-S500" />
 	<!-- right shoulder pitch 1 link -->
         <link name="r_arm_sh_p1_link">
@@ -358,8 +368,9 @@
           <parent link="r_arm_sh_p1_link"/>
           <child link="r_arm_sh_r_link"/>
-          <limit velocity="6.5" effort="1000" lower="${-pi*0.5}" upper="${pi*0.3}" />
-          <dynamics damping="0.1" friction="0.1" />
-        </joint>
-        <xacro:insert_transmission name="r_arm_sh_r" />
+          <!--limit velocity="6.5" effort="1000" lower="${-pi*0.5}" upper="${pi*0.3}" />
+          <dynamics damping="0.1" friction="0.1" /-->
+	  <xacro:joint_medium_servo_limits_macro lower="${-pi*0.5}" upper="${pi*0.3}" />
+        </joint>
+        <xacro:effort_transmission name="r_arm_sh_r" servo="H54-100-S500" />
 	<!-- right shoulder roll link -->
         <link name="r_arm_sh_r_link">
@@ -390,8 +401,9 @@
           <parent link="r_arm_sh_r_link"/>
           <child link="r_arm_sh_p2_link"/>
-          <limit velocity="6.5" effort="1000" lower="${-pi*0.5}" upper="${pi*0.5}" />
-          <dynamics damping="0.1" friction="0.1" />
-        </joint>
-        <xacro:insert_transmission name="r_arm_sh_p2" />
+          <!--limit velocity="6.5" effort="1000" lower="${-pi*0.5}" upper="${pi*0.5}" />
+          <dynamics damping="0.1" friction="0.1" /-->
+	  <xacro:joint_medium_servo_limits_macro lower="${-pi*0.5}" upper="${pi*0.5}" />
+        </joint>
+        <xacro:effort_transmission name="r_arm_sh_p2" servo="H54-100-S500" />
 	<!-- right shoulder pitch2 link -->
         <link name="r_arm_sh_p2_link">
@@ -422,8 +434,9 @@
           <parent link="r_arm_sh_p2_link"/>
           <child link="r_arm_el_y_link"/>
-          <limit velocity="6.5" effort="1000" lower="${-pi*0.4}" upper="${pi*0.4}" />
-          <dynamics damping="0.1" friction="0.1" />
-        </joint>
-        <xacro:insert_transmission name="r_arm_el_y" />
+          <!--limit velocity="6.5" effort="1000" lower="${-pi*0.4}" upper="${pi*0.4}" />
+          <dynamics damping="0.1" friction="0.1" /-->
+	  <xacro:joint_medium_servo_limits_macro lower="${-pi*0.4}" upper="${pi*0.4}" />
+        </joint>
+        <xacro:effort_transmission name="r_arm_el_y" servo="H54-100-S500" />
 	<!-- right elbow yaw link -->
         <link name="r_arm_el_y_link">
@@ -454,8 +467,9 @@
           <parent link="r_arm_el_y_link"/>
           <child link="r_arm_wr_r_link"/>
-          <limit velocity="6.5" effort="1000" lower="${-pi*0.5}" upper="${pi*0.5}" />
-          <dynamics damping="0.1" friction="0.1" />
-        </joint>
-        <xacro:insert_transmission name="r_arm_wr_r" />
+          <!--limit velocity="6.5" effort="1000" lower="${-pi*0.5}" upper="${pi*0.5}" />
+          <dynamics damping="0.1" friction="0.1" /-->
+	  <xacro:joint_small_servo_limits_macro lower="${-pi*0.5}" upper="${pi*0.5}" />
+        </joint>
+        <xacro:effort_transmission name="r_arm_wr_r" servo="H42-20-S300" />
 	<!-- right wrist roll link -->
         <link name="r_arm_wr_r_link">
@@ -486,8 +500,9 @@
           <parent link="r_arm_wr_r_link"/>
           <child link="r_arm_wr_y_link"/>
-          <limit velocity="6.5" effort="1000" lower="${-pi*0.45}" upper="${pi*0.45}" />
-          <dynamics damping="0.1" friction="0.1" />
-        </joint>
-        <xacro:insert_transmission name="r_arm_wr_y" />
+          <!--limit velocity="6.5" effort="1000" lower="${-pi*0.45}" upper="${pi*0.45}" />
+          <dynamics damping="0.1" friction="0.1" /-->
+	  <xacro:joint_small_servo_limits_macro lower="${-pi*0.45}" upper="${pi*0.45}" />
+        </joint>
+        <xacro:effort_transmission name="r_arm_wr_y" servo="H42-20-S300" />
 	<!-- right wrist yaw link -->
         <link name="r_arm_wr_y_link">
@@ -518,8 +533,9 @@
           <parent link="r_arm_wr_y_link"/>
           <child link="r_arm_wr_p_link"/>
-          <limit velocity="6.5" effort="1000" lower="${-pi*0.45}" upper="${pi*0.45}" />
-          <dynamics damping="0.1" friction="0.1" />
-        </joint>
-        <xacro:insert_transmission name="r_arm_wr_p" />
+          <!--limit velocity="6.5" effort="1000" lower="${-pi*0.45}" upper="${pi*0.45}" />
+          <dynamics damping="0.1" friction="0.1" /-->
+	  <xacro:joint_small_servo_limits_macro lower="${-pi*0.45}" upper="${pi*0.45}" />
+        </joint>
+        <xacro:effort_transmission name="r_arm_wr_p" servo="H42-20-S300" />
 	<!-- right wrist pitch link -->
         <link name="r_arm_wr_p_link">
@@ -550,8 +566,9 @@
           <parent link="r_arm_wr_p_link"/>
           <child link="r_arm_grip_link"/>
-          <limit velocity="6.5" effort="1000" lower="${-pi*0.45}" upper="${pi*0.45}" />
-          <dynamics damping="0.1" friction="0.1" />
-        </joint>
-        <xacro:insert_transmission name="r_arm_grip" />
+          <!--limit velocity="6.5" effort="1000" lower="${-pi*0.45}" upper="${pi*0.45}" />
+          <dynamics damping="0.1" friction="0.1" /-->
+	  <xacro:joint_small_servo_limits_macro lower="${-pi*0.45}" upper="${pi*0.45}" />
+        </joint>
+        <xacro:effort_transmission name="r_arm_grip" servo="H42-20-S300" />
 	<!-- right arm gripper link -->
         <link name="r_arm_grip_link">
@@ -582,8 +599,9 @@
           <parent link="r_arm_wr_p_link"/>
           <child link="r_arm_grip_1_link"/>
-          <limit velocity="6.5" effort="1000" lower="${-pi*0.45}" upper="${pi*0.45}" />
-          <dynamics damping="0.1" friction="0.1" />
-        </joint>
-        <xacro:insert_transmission name="r_arm_grip_1" />
+          <!--limit velocity="6.5" effort="1000" lower="${-pi*0.45}" upper="${pi*0.45}" />
+          <dynamics damping="0.1" friction="0.1" /-->
+	  <xacro:joint_small_servo_limits_macro lower="${-pi*0.45}" upper="${pi*0.45}" />
+        </joint>
+        <xacro:effort_transmission name="r_arm_grip_1" servo="H42-20-S300" />
 	<!-- right arm gripper link -->
         <link name="r_arm_grip_1_link">

File: robotis_humanoid_description/urdf/robotis_humanoid.structure.head.xacro (robot description, xacro)
@@ -9,8 +9,9 @@
           <parent link="${parent}"/>
           <child link="head_y_link"/>
-          <limit velocity="6.5" effort="1000" lower="${-pi*0.5}" upper="${pi*0.5}" />
-          <dynamics damping="0.1" friction="0.1" />
+          <!--limit velocity="6.5" effort="1000" lower="${-pi*0.5}" upper="${pi*0.5}" />
+          <dynamics damping="0.1" friction="0.1" /-->
+	  <xacro:joint_small_servo_limits_macro lower="${-pi*0.5}" upper="${pi*0.5}" />
         </joint>
-        <xacro:insert_transmission name="head_y" />
+        <xacro:effort_transmission name="head_y" servo="H42-20-S300" />
 	<!-- head yaw link -->
         <link name="head_y_link">
@@ -36,8 +37,9 @@
           <parent link="head_y_link"/>
           <child link="head_p_link"/>
-          <limit velocity="6.5" effort="1000" lower="${-pi*0.5}" upper="${pi*0.5}" />
-          <dynamics damping="0.1" friction="0.1" />
+          <!--limit velocity="6.5" effort="1000" lower="${-pi*0.5}" upper="${pi*0.5}" />
+          <dynamics damping="0.1" friction="0.1" /-->
+	  <xacro:joint_small_servo_limits_macro lower="${-pi*0.5}" upper="${pi*0.5}" />
         </joint>
-        <xacro:insert_transmission name="head_p" />
+        <xacro:effort_transmission name="head_p" servo="H42-20-S300" />
 	<!-- head pitch link -->
         <link name="head_p_link">
