Commit message: added motor-models and transmission-names

File: robotis_humanoid_description/urdf/robotis_humanoid.structure.leg.xacro (robot description, xacro)
@@ -9,8 +9,9 @@
           <parent link="${parent}"/>
           <child link="l_leg_hip_y_link"/>
-          <limit velocity="6.5" effort="1000" lower="${-pi*0.45}" upper="${pi*0.45}" />
-          <dynamics damping="0.1" friction="0.1" />
-        </joint>
-        <xacro:insert_transmission name="l_leg_hip_y" />
+          <!--limit velocity="6.5" effort="1000" lower="${-pi*0.45}" upper="${pi*0.45}" />
+          <dynamics damping="0.1" friction="0.1" /-->
+	  <xacro:joint_medium_servo_limits_macro lower="${-pi*0.45}" upper="${pi*0.45}" />
+        </joint>
+        <xacro:effort_transmission name="l_leg_hip_y" servo="H54-100-S500" />
 	<!-- left hip yaw link -->
         <link name="l_leg_hip_y_link">
@@ -41,8 +42,9 @@
           <parent link="l_leg_hip_y_link"/>
           <child link="l_leg_hip_r_link"/>
-          <limit velocity="6.5" effort="1000" lower="${-pi*0.2}" upper="${pi*0.3}" />
-          <dynamics damping="0.1" friction="0.1" />
-        </joint>
-        <xacro:insert_transmission name="l_leg_hip_r" />
+          <!--limit velocity="6.5" effort="1000" lower="${-pi*0.2}" upper="${pi*0.3}" />
+          <dynamics damping="0.1" friction="0.1" /-->
+	  <xacro:joint_large_servo_limits_macro lower="${-pi*0.2}" upper="${pi*0.3}" />
+        </joint>
+        <xacro:effort_transmission name="l_leg_hip_r" servo="H54-200-S500" />
 	<!-- left hip roll link -->
         <link name="l_leg_hip_r_link">
@@ -73,8 +75,9 @@
           <parent link="l_leg_hip_r_link"/>
           <child link="l_leg_hip_p_link"/>
-          <limit velocity="6.5" effort="1000" lower="${-pi*0.4}" upper="${pi*0.4}" />
-          <dynamics damping="0.1" friction="0.1" />
-        </joint>
-        <xacro:insert_transmission name="l_leg_hip_p" />
+          <!--limit velocity="6.5" effort="1000" lower="${-pi*0.4}" upper="${pi*0.4}" />
+          <dynamics damping="0.1" friction="0.1" /-->
+	  <xacro:joint_large_servo_limits_macro lower="${-pi*0.4}" upper="${pi*0.4}" />
+        </joint>
+        <xacro:effort_transmission name="l_leg_hip_p" servo="H54-200-S500" />
 	<!-- left hip pitch link -->
         <link name="l_leg_hip_p_link">
@@ -105,8 +108,9 @@
           <parent link="l_leg_hip_p_link"/>
           <child link="l_leg_kn_p_link"/>
-          <limit velocity="6.5" effort="1000" lower="${-pi*0.1}" upper="${pi*0.7}" />
-          <dynamics damping="0.1" friction="0.1" />
-        </joint>
-        <xacro:insert_transmission name="l_leg_kn_p" />
+          <!--limit velocity="6.5" effort="1000" lower="${-pi*0.1}" upper="${pi*0.7}" />
+          <dynamics damping="0.1" friction="0.1" /-->
+	  <xacro:joint_large_servo_limits_macro lower="${-pi*0.1}" upper="${pi*0.7}" />
+        </joint>
+        <xacro:effort_transmission name="l_leg_kn_p" servo="H54-200-S500" />
 	<!-- left knee pitch link -->
         <link name="l_leg_kn_p_link">
@@ -137,8 +141,9 @@
           <parent link="l_leg_kn_p_link"/>
           <child link="l_leg_an_p_link"/>
-          <limit velocity="6.5" effort="1000" lower="${-pi*0.45}" upper="${pi*0.45}" />
-          <dynamics damping="0.1" friction="0.1" />
-        </joint>
-        <xacro:insert_transmission name="l_leg_an_p" />
+          <!--limit velocity="6.5" effort="1000" lower="${-pi*0.45}" upper="${pi*0.45}" />
+          <dynamics damping="0.1" friction="0.1" /-->
+	  <xacro:joint_large_servo_limits_macro lower="${-pi*0.45}" upper="${pi*0.45}" />
+        </joint>
+        <xacro:effort_transmission name="l_leg_an_p" servo="H54-200-S500" />
 	<!-- left ankle pitch link -->
         <link name="l_leg_an_p_link">
@@ -169,8 +174,9 @@
           <parent link="l_leg_an_p_link"/>
           <child link="l_leg_an_r_link"/>
-          <limit velocity="6.5" effort="1000" lower="${-pi*0.5}" upper="${pi*0.4}" />
-          <dynamics damping="0.1" friction="0.1" />
-        </joint>
-        <xacro:insert_transmission name="l_leg_an_r" />
+          <!--limit velocity="6.5" effort="1000" lower="${-pi*0.5}" upper="${pi*0.4}" />
+          <dynamics damping="0.1" friction="0.1" /-->
+	  <xacro:joint_large_servo_limits_macro lower="${-pi*0.5}" upper="${pi*0.4}" />
+        </joint>
+        <xacro:effort_transmission name="l_leg_an_r" servo="H54-200-S500" />
 	<!-- left ankle roll link -->
         <link name="l_leg_an_r_link">
@@ -231,8 +237,9 @@
           <parent link="${parent}"/>
           <child link="r_leg_hip_y_link"/>
-          <limit velocity="6.5" effort="1000" lower="${-pi*0.45}" upper="${pi*0.45}" />
-          <dynamics damping="0.1" friction="0.1" />
-        </joint>
-        <xacro:insert_transmission name="r_leg_hip_y" />
+          <!--limit velocity="6.5" effort="1000" lower="${-pi*0.45}" upper="${pi*0.45}" />
+          <dynamics damping="0.1" friction="0.1" /-->
+	  <xacro:joint_medium_servo_limits_macro lower="${-pi*0.45}" upper="${pi*0.45}" />
+        </joint>
+        <xacro:effort_transmission name="r_leg_hip_y" servo="H54-100-S500" />
 	<!-- right hip yaw link -->
         <link name="r_leg_hip_y_link">
@@ -263,8 +270,9 @@
           <parent link="r_leg_hip_y_link"/>
           <child link="r_leg_hip_r_link"/>
-          <limit velocity="6.5" effort="1000" lower="${-pi*0.3}" upper="${pi*0.2}" />
-          <dynamics damping="0.1" friction="0.1" />
-        </joint>
-        <xacro:insert_transmission name="r_leg_hip_r" />
+          <!--limit velocity="6.5" effort="1000" lower="${-pi*0.3}" upper="${pi*0.2}" />
+          <dynamics damping="0.1" friction="0.1" /-->
+	  <xacro:joint_large_servo_limits_macro lower="${-pi*0.3}" upper="${pi*0.2}" />
+        </joint>
+        <xacro:effort_transmission name="r_leg_hip_r" servo="H54-200-S500" />
 	<!-- right hip roll link -->
         <link name="r_leg_hip_r_link">
@@ -295,8 +303,9 @@
           <parent link="r_leg_hip_r_link"/>
           <child link="r_leg_hip_p_link"/>
-          <limit velocity="6.5" effort="1000" lower="${-pi*0.4}" upper="${pi*0.4}" />
-          <dynamics damping="0.1" friction="0.1" />
-        </joint>
-        <xacro:insert_transmission name="r_leg_hip_p" />
+          <!--limit velocity="6.5" effort="1000" lower="${-pi*0.4}" upper="${pi*0.4}" />
+          <dynamics damping="0.1" friction="0.1" /-->
+	  <xacro:joint_large_servo_limits_macro lower="${-pi*0.4}" upper="${pi*0.4}" />
+        </joint>
+        <xacro:effort_transmission name="r_leg_hip_p" servo="H54-200-S500" />
 	<!-- right hip pitch link -->
         <link name="r_leg_hip_p_link">
@@ -327,8 +336,9 @@
           <parent link="r_leg_hip_p_link"/>
           <child link="r_leg_kn_p_link"/>
-          <limit velocity="6.5" effort="1000" lower="${-pi*0.7}" upper="${pi*0.1}" />
-          <dynamics damping="0.1" friction="0.1" />
-        </joint>
-        <xacro:insert_transmission name="r_leg_kn_p" />
+          <!--limit velocity="6.5" effort="1000" lower="${-pi*0.7}" upper="${pi*0.1}" />
+          <dynamics damping="0.1" friction="0.1" /-->
+	  <xacro:joint_large_servo_limits_macro lower="${-pi*0.7}" upper="${pi*0.1}" />
+        </joint>
+        <xacro:effort_transmission name="r_leg_kn_p" servo="H54-200-S500" />
 	<!-- right knee pitch link -->
         <link name="r_leg_kn_p_link">
@@ -359,8 +369,9 @@
           <parent link="r_leg_kn_p_link"/>
           <child link="r_leg_an_p_link"/>
-          <limit velocity="6.5" effort="1000" lower="${-pi*0.45}" upper="${pi*0.45}" />
-          <dynamics damping="0.1" friction="0.1" />
-        </joint>
-        <xacro:insert_transmission name="r_leg_an_p" />
+          <!--limit velocity="6.5" effort="1000" lower="${-pi*0.45}" upper="${pi*0.45}" />
+          <dynamics damping="0.1" friction="0.1" /-->
+	  <xacro:joint_large_servo_limits_macro lower="${-pi*0.45}" upper="${pi*0.45}" />
+        </joint>
+        <xacro:effort_transmission name="r_leg_an_p" servo="H54-200-S500" />
 	<!-- right ankle pitch link -->
         <link name="r_leg_an_p_link">
@@ -391,8 +402,9 @@
           <parent link="r_leg_an_p_link"/>
           <child link="r_leg_an_r_link"/>
-          <limit velocity="6.5" effort="1000" lower="${-pi*0.45}" upper="${pi*0.45}" />
-          <dynamics damping="0.1" friction="0.1" />
-        </joint>
-        <xacro:insert_transmission name="r_leg_an_r" />
+          <!--limit velocity="6.5" effort="1000" lower="${-pi*0.45}" upper="${pi*0.45}" />
+          <dynamics damping="0.1" friction="0.1" /-->
+	  <xacro:joint_large_servo_limits_macro lower="${-pi*0.45}" upper="${pi*0.45}" />
+        </joint>
+        <xacro:effort_transmission name="r_leg_an_r" servo="H54-200-S500" />
 	<!-- right ankle roll link -->
         <link name="r_leg_an_r_link">

File: robotis_humanoid_description/urdf/robotis_humanoid.transmissions.xacro (robot description, xacro)
@@ -1,5 +1,5 @@
 <?xml version="1.0"?>
 <robot xmlns:xacro="http://ros.org/wiki/xacro">
-	<xacro:macro name="insert_transmission" params="name">
+	<xacro:macro name="effort_transmission" params="name servo">
 		<transmission name="${name}_tran">
 			<type>transmission_interface/SimpleTransmission</type>
@@ -7,5 +7,5 @@
 				<hardwareInterface>EffortJointInterface</hardwareInterface>
 			</joint>
-			<actuator name="${name}_motor">
+			<actuator name="${name}_${servo}_motor">
 				<hardwareInterface>EffortJointInterface</hardwareInterface>
 				<mechanicalReduction>1</mechanicalReduction>
@@ -13,3 +13,15 @@
 		</transmission>
 	</xacro:macro>
+	<xacro:macro name="position_transmission" params="name servo">
+		<transmission name="${name}_tran">
+			<type>transmission_interface/SimpleTransmission</type>
+			<joint name="${name}">
+				<hardwareInterface>PositionJointInterface</hardwareInterface>
+			</joint>
+			<actuator name="${name}_${servo}_motor">
+				<hardwareInterface>PositionJointInterface</hardwareInterface>
+				<mechanicalReduction>1</mechanicalReduction>
+			</actuator>
+		</transmission>
+	</xacro:macro>
 </robot>

File: robotis_humanoid_description/urdf/robotis_humanoid.xacro (robot description, xacro)
@@ -13,4 +13,5 @@
   <xacro:include filename="$(find robotis_humanoid_description)/urdf/robotis_humanoid.inertia.xacro" />
   <xacro:include filename="$(find robotis_humanoid_description)/urdf/robotis_humanoid.transmissions.xacro" />
+  <xacro:include filename="$(find robotis_humanoid_description)/urdf/servos.xacro" />
   <!-- Used for fixing robot -->
 <!--
@@ -58,8 +59,9 @@
     <origin xyz="0 0 0.1705" rpy="0 0 0"/>
     <axis xyz="0 0 1"/>
-    <limit velocity="6.5" effort="1000" lower="${-pi*0.6}" upper="${pi*0.6}" />
-    <dynamics damping="0.1" friction="0.1" />
+    <!--limit velocity="6.5" effort="1000" lower="${-pi*0.6}" upper="${pi*0.6}" />
+    <dynamics damping="0.1" friction="0.1" /-->
+    <xacro:joint_medium_servo_limits_macro lower="${-pi*0.6}" upper="${pi*0.6}" />
   </joint>
-  <xacro:insert_transmission name="torso_y" />
+  <xacro:effort_transmission name="torso_y" servo="H54-100-S500" />
   <!-- chest_link -->
   <link name="chest_link">

Commit message: integrated vt hands

File: robotis_humanoid_description/urdf/robotis_humanoid.structure.arm.xacro (robot description, xacro)
@@ -206,111 +206,28 @@
         </joint>
         <xacro:position_transmission name="${prefix}_arm_wr_p" servo="H42-20-S300" />
-	<!-- wrist pitch link -->
-        <link name="${prefix}_arm_wr_p_link">
-    	  <collision>
-      	    <origin xyz="0 0 0" rpy="0 0 0"/>
-      	    <geometry>
-              <box size="0.01 0.01 0.01" />
-      	    </geometry>
-    	  </collision>
-   	  <visual>
-      	    <origin xyz="0 0 0" rpy="0 0 0"/>
-      	    <geometry>
-              <mesh filename="package://robotis_humanoid_description/meshes/robotis_${prefix}_arm_wr_p_link.stl" scale="0.001 0.001 0.001"/>
-      	    </geometry>
-      	    <material name="grey"/>
-    	  </visual>
-          <inertial>
-      	    <origin xyz="0.065 ${reflect*0.045} 0.000" rpy="0 0 0"/>
-      	    <mass value="0.565"/>
-            <inertia ixx="0.00047" ixy="${reflect*-0.00001}" ixz="0.0" iyy="0.00042" iyz="0.0" izz="0.00058" />
-    	  </inertial>
-        </link>
-	<!-- arm gripper -->
-<!--
-        <joint name="${prefix}_arm_grip" type="revolute">
-          <axis xyz="0 0 1" />
-          <origin xyz="0.0877 ${reflect*0.0583} 0.0" rpy="0 0 0"/>
-          <parent link="${prefix}_arm_wr_p_link"/>
-          <child link="${prefix}_arm_grip_link"/>
-          <limit velocity="6.5" effort="1000" lower="${-pi*0.45}" upper="${pi*0.45}" />
-          <dynamics damping="0.1" friction="0.1" />
-        </joint>
-        <xacro:position_transmission name="${prefix}_arm_grip" servo="H42-20-S300" />
-        <link name="${prefix}_arm_grip_link">
-    	  <collision>
-      	    <origin xyz="0 0 0" rpy="0 0 0"/>
-      	    <geometry>
-              <box size="0.01 0.01 0.01" />
-      	    </geometry>
-    	  </collision>
-   	  <visual>
-      	    <origin xyz="0 0 0" rpy="0 0 0"/>
-      	    <geometry>
-              <mesh filename="package://robotis_humanoid_description/meshes/robotis_${prefix}_arm_grip_link.stl" scale="0.001 0.001 0.001"/>
-      	    </geometry>
-      	    <material name="grey"/>
-    	  </visual>
-          <inertial>
-      	    <origin xyz="0.031 ${reflect*0.014} 0.000" rpy="0 0 0"/>
-      	    <mass value="0.013"/>
-            <inertia ixx="0.0" ixy="0.0" ixz="0.0" iyy="0.00001" iyz="0.0" izz="0.00001" />
-    	  </inertial>
-        </link>
-        <joint name="${prefix}_arm_grip_1" type="revolute">
-          <axis xyz="0 0 1" />
-          <origin xyz="0.0877 ${reflect*0.0317} 0.0" rpy="0 0 0"/>
-          <parent link="${prefix}_arm_wr_p_link"/>
-          <child link="${prefix}_arm_grip_1_link"/>
-          <limit velocity="6.5" effort="1000" lower="${-pi*0.45}" upper="${pi*0.45}" />
-          <dynamics damping="0.1" friction="0.1" />
-        </joint>
-        <xacro:position_transmission name="${prefix}_arm_grip_1" servo="H42-20-S300" />
-        <link name="${prefix}_arm_grip_1_link">
-    	  <collision>
-      	    <origin xyz="0 0 0" rpy="0 0 0"/>
-      	    <geometry>
-              <box size="0.01 0.01 0.01" />
-      	    </geometry>
-    	  </collision>
-   	  <visual>
-      	    <origin xyz="0 0 0" rpy="0 0 0"/>
-      	    <geometry>
-              <mesh filename="package://robotis_humanoid_description/meshes/robotis_${prefix}_arm_grip_1_link.stl" scale="0.001 0.001 0.001"/>
-      	    </geometry>
-      	    <material name="grey"/>
-    	  </visual>
-          <inertial>
-      	    <origin xyz="0.031 ${reflect*-0.014} 0.000" rpy="0 0 0"/>
-      	    <mass value="0.013"/>
-            <inertia ixx="0.0" ixy="0.0" ixz="0.0" iyy="0.00001" iyz="0.0" izz="0.00001" />
-    	  </inertial>
-        </link>
-        <joint name="${prefix}_arm_end" type="fixed">
-          <origin xyz="0.145 ${reflect*0.045} 0" rpy="0 0 0"/>
-          <parent link="${prefix}_arm_wr_p_link"/>
-          <child link="${prefix}_arm_end_link"/>
-        </joint>
-        <link name="${prefix}_arm_end_link">
-    	  <collision>
-      	    <origin xyz="0 0 0" rpy="0 0 0"/>
-      	    <geometry>
-              <box size="0.01 0.01 0.01" />
-      	    </geometry>
-    	  </collision>
-   	  <visual>
-      	    <origin xyz="0 0 0" rpy="0 0 0"/>
-      	    <geometry>
-              <box size="0.01 0.01 0.01" />
-      	    </geometry>
-      	    <material name="red"/>
-    	  </visual>
-          <inertial>
-      	    <origin xyz="0.0 0.0 0.0" rpy="0 0 0"/>
-      	    <mass value="0.001"/>
-      	    <inertia ixx="0.00001" ixy="0.0" ixz="0.0" iyy="0.00001" iyz="0.0" izz="0.00001" />
-    	  </inertial>
-        </link>
--->
+  <link name="${prefix}_arm_wr_p_link">
+    <xacro:inertial_sphere_with_pose_macro mass="0.27" diameter="0.03">
+      <origin xyz="0.0 0.0 -0.03" rpy="0 0 0"/>
+    </xacro:inertial_sphere_with_pose_macro>
+    <visual>
+      <origin
+        xyz="0 ${reflect*0.042} 0"
+        rpy="0 ${pi*0.5} ${pi*0.5}" />
+      <geometry>
+        <mesh
+          filename="package://thor_mang_description/meshes/visual/wrist_roll.stl" scale="${-0.001 * reflect} 0.001 0.001"/>
+      </geometry>
+      <xacro:black/>
+    </visual>
+    <collision>
+      <origin
+        xyz="0 ${reflect*0.042} 0"
+        rpy="0 ${pi*0.5} ${pi*0.5}" />
+      <geometry>
+        <mesh
+          filename="package://thor_mang_description/meshes/visual/wrist_roll.stl" scale="${-0.001 * reflect} 0.001 0.001"/>
+      </geometry>
+    </collision>
+  </link>
     </xacro:macro>
 </robot>

File: robotis_humanoid_description/urdf/robotis_humanoid.transmissions.xacro (robot description, xacro)
@@ -17,8 +17,20 @@
 			<type>transmission_interface/SimpleTransmission</type>
 			<joint name="${name}">
-				<hardwareInterface>EffortJointInterface</hardwareInterface>
+				<hardwareInterface>PositionJointInterface</hardwareInterface>
 			</joint>
 			<actuator name="${servo}_motor">
-				<hardwareInterface>EffortJointInterface</hardwareInterface>
+				<hardwareInterface>PositionJointInterface</hardwareInterface>
+				<mechanicalReduction>1</mechanicalReduction>
+			</actuator>
+		</transmission>
+	</xacro:macro>
+	<xacro:macro name="velocity_transmission" params="name servo">
+		<transmission name="${name}_tran">
+			<type>transmission_interface/SimpleTransmission</type>
+			<joint name="${name}">
+				<hardwareInterface>VelocityJointInterface</hardwareInterface>
+			</joint>
+			<actuator name="${servo}_motor">
+				<hardwareInterface>VelocityJointInterface</hardwareInterface>
 				<mechanicalReduction>1</mechanicalReduction>
 			</actuator>

File: robotis_humanoid_description/urdf/robotis_humanoid.xacro (robot description, xacro)
@@ -1,4 +1,3 @@
 <?xml version="1.0"?>
-<!-- Revolute-Revolute Manipulator -->
 <robot name="robotis_humanoid" xmlns:xacro="http://www.ros.org/wiki/xacro">
   <!-- some parameters -->
@@ -15,4 +14,5 @@
   <xacro:include filename="$(find robotis_humanoid_description)/urdf/robotis_humanoid.transmissions.xacro" />
   <xacro:include filename="$(find robotis_humanoid_description)/urdf/servos.xacro" />
+<macro name="robotis_humanoid_macro">
   <!-- Used for fixing robot -->
   <link name="world">
@@ -38,5 +38,5 @@
     arm_joint_2_limit_lower="${-pi*0.3}"
     arm_joint_2_limit_upper="${pi*0.5}"
-      arm_joint_3_limit_lower="${-pi*0.5}"
+    arm_joint_3_limit_lower="${-pi*0.5}"
     arm_joint_3_limit_upper="${pi*0.5}"
     arm_joint_4_limit_lower="${-pi*0.4}"
@@ -100,3 +100,4 @@
   />
   <xacro:robotis_humanoid_head parent="chest_link" />
+</macro>
 </robot>
